File: prototype/output/pcbs/board.kicad_pcb (KiCad board)
At the start: 2 copper layers, 157.8 x 123.9 mm, 46 parts

Commit message: latest pcb
Parts:
- moved D19 4.63 mm to (99.2, 23.8), turned to -20 degrees
- moved S19 4.47 mm to (97.5, 28.5), turned to 160 degrees
- moved D20 4.13 mm to (118.3, 32.4), turned to -26 degrees
- moved S20 4.03 mm to (116.1, 36.9), turned to 154 degrees
Other:
- board size 157.8 x 123.9 mm -> 157.8 x 119.6 mm
